Commit message: Simplify urdf files. Add node_test.py for testing image and joint state topics

File: urdf/binocular_laser_profile_scanner.xacro (robot description, xacro)
@@ -1,5 +1,7 @@
 <?xml version="1.0" encoding="utf-8"?>
 <robot xmlns:xacro="http://www.ros.org/wiki/xacro" name="binocular_laser_profile_scanner">
-  <xacro:include filename="$(find binocular_laser_profile_scanner)/urdf/gazebo_camera_plugin.xacro"/>
+  <xacro:include filename="$(find binocular_laser_profile_scanner)/urdf/gazebo_camera.xacro"/>
+  <xacro:include filename="$(find binocular_laser_profile_scanner)/urdf/gazebo_projector.xacro"/>
+  <xacro:include filename="$(find binocular_laser_profile_scanner)/urdf/gazebo_controller.xacro"/>
   <link name="world"/>
   <joint name="world_joint" type="fixed">
@@ -434,67 +436,3 @@
       xyz="0 0 0" />
   </joint>
-  <!-- projector deneme v1
-  <gazebo reference="line_laser_link">
-    <material>Gazebo/Red</material>
-    <projector name="line_projector">
-      <pose> 0 0 0 0 0 0 </pose>
-      <texture>building_frame.png</texture>
-      <near_clip>0.01</near_clip>
-      <far_clip>10.0</far_clip>
-      <fov>0.1</fov>
-      <plugin name="projector_controller" filename="libgazebo_ros_projector.so">
-        <update_rate>10.0</update_rate>
-      </plugin>
-    </projector>
-  </gazebo>
-  -->
-  <gazebo reference="line_laser_link">
-    <projector name="projector">
-      <pose>0 0 0 0 ${pi} 0</pose>
-      <texture>line_laser.png</texture>
-      <fov>2.0</fov>
-      <near_clip>0.005</near_clip>
-      <far_clip>1.0</far_clip>
-    </projector>
-  </gazebo>
-  <gazebo>
-    <plugin name="projector_controller" filename="libgazebo_ros_projector.so">
-      <projector>line_laser_link/projector</projector>
-      <alwaysOn>true</alwaysOn>
-      <updateRate>15.0</updateRate>
-      <textureName>line_laser_5p.png</textureName>
-      <textureTopicName>projector_controller/image</textureTopicName>
-      <projectorTopicName>projector_controller/projector</projectorTopicName>
-    </plugin>
-  </gazebo>
-  <!-- Line Laser Projector -->
-  <!--
-  <xacro:include filename="$(find binocular_laser_profile_scanner)/urdf/gazebo_projector.xacro"/>
-  -->
-  <gazebo>
-    <plugin name="gazebo_ros_control" filename="libgazebo_ros_control.so">
-      <robotNamespace>/binocular_laser_profile_scanner</robotNamespace>
-      <robotSimType>gazebo_ros_control/DefaultRobotHWSim</robotSimType>
-    </plugin>
-  </gazebo>
-  <transmission name="tran1">
-    <type>transmission_interface/SimpleTransmission</type>
-    <joint name="rot_table_joint">
-      <hardwareInterface>hardware_interface/EffortJointInterface</hardwareInterface>
-    </joint>
-    <actuator name="rot_table_motor">
-      <hardwareInterface>hardware_interface/EffortJointInterface</hardwareInterface>
-      <mechanicalReduction>1</mechanicalReduction>
-    </actuator>
-  </transmission>
-   <transmission name="tran2">
-    <type>transmission_interface/SimpleTransmission</type>
-    <joint name="motor_joint">
-      <hardwareInterface>hardware_interface/EffortJointInterface</hardwareInterface>
-    </joint>
-    <actuator name="scanner_angle_motor">
-      <hardwareInterface>hardware_interface/EffortJointInterface</hardwareInterface>
-      <mechanicalReduction>1</mechanicalReduction>
-    </actuator>
-  </transmission>
 </robot>

File: urdf/gazebo_camera.xacro (robot description, xacro)
@@ -4,6 +4,4 @@
     CHANGES
     * Pixel numbers of image sensor reduced to 600 px x 600 px due to low fps
-    * Image grabbing mode changed from continuous to software trigger
-      in order to prevent shifting between calculated distance and real distance
     Image Sensor Specs used before
     Sensor: IMX548

File: urdf/gazebo_projector.xacro (robot description, xacro)
@@ -1,16 +1,22 @@
-<?xml version="1.0"?>
-<robot xmlns:xacro="http://www.ros.org/wiki/xacro">
-    <gazebo reference="line_laser_link">
-        <material>Gazebo/Red</material>
-        <projector name="line_projector">
-            <pose> 0 0 0 0 0 0 </pose>
-            <texture>building_frame.png</texture>
-            <near_clip>0.01</near_clip>
-            <far_clip>10.0</far_clip>
-            <fov>0.5</fov>
-            <plugin name="projector_controller" filename="libgazebo_ros_projector.so">
-                <update_rate>10.0</update_rate>
-            </plugin>
-        </projector>
-    </gazebo>
+<?xml version="1.0" encoding="utf-8"?>
 <robot>
+  <gazebo reference="line_laser_link">
+    <projector name="projector">
+      <pose>0 0 0 0 ${pi} 0</pose>
+      <texture>line_laser.png</texture>
+      <fov>2.0</fov>
+      <near_clip>0.005</near_clip>
+      <far_clip>1.0</far_clip>
+    </projector>
+  </gazebo>
+  <gazebo>
+    <plugin name="projector_controller" filename="libgazebo_ros_projector.so">
+      <projector>line_laser_link/projector</projector>
+      <alwaysOn>true</alwaysOn>
+      <updateRate>15.0</updateRate>
+      <textureName>line_laser.png</textureName>
+      <textureTopicName>projector_controller/image</textureTopicName>
+      <projectorTopicName>projector_controller/projector</projectorTopicName>
+    </plugin>
+  </gazebo>
+</robot>

Commit message: initial commit

File: urdf/binocular_laser_profile_scanner.xacro (robot description, xacro)
@@ -32,19 +32,19 @@
       <geometry>
         <mesh
-          filename="package://binocular_laser_profile_scanner/meshes/base_link.STL" />
-      </geometry>
-      <material
-        name="">
-        <color
-          rgba="0.792156862745098 0.819607843137255 0.933333333333333 1" />
-      </material>
-    </visual>
-    <collision>
-      <origin
-        xyz="0 0 0"
-        rpy="0 0 0" />
-      <geometry>
-        <mesh
-          filename="package://binocular_laser_profile_scanner/meshes/base_link.STL" />
+          filename="file://$(find binocular_laser_profile_scanner)/meshes/base_link.STL" />
+      </geometry>
+      <material
+        name="">
+        <color
+          rgba="0.792156862745098 0.819607843137255 0.933333333333333 1" />
+      </material>
+    </visual>
+    <collision>
+      <origin
+        xyz="0 0 0"
+        rpy="0 0 0" />
+      <geometry>
+        <mesh
+          filename="file://$(find binocular_laser_profile_scanner)/meshes/base_link.STL" />
       </geometry>
     </collision>
@@ -72,19 +72,19 @@
       <geometry>
         <mesh
-          filename="package://binocular_laser_profile_scanner/meshes/rot_table_link.STL" />
-      </geometry>
-      <material
-        name="">
-        <color
-          rgba="0.792156862745098 0.819607843137255 0.933333333333333 1" />
-      </material>
-    </visual>
-    <collision>
-      <origin
-        xyz="0 0 0"
-        rpy="0 0 0" />
-      <geometry>
-        <mesh
-          filename="package://binocular_laser_profile_scanner/meshes/rot_table_link.STL" />
+          filename="file://$(find binocular_laser_profile_scanner)/meshes/rot_table_link.STL" />
+      </geometry>
+      <material
+        name="">
+        <color
+          rgba="0.792156862745098 0.819607843137255 0.933333333333333 1" />
+      </material>
+    </visual>
+    <collision>
+      <origin
+        xyz="0 0 0"
+        rpy="0 0 0" />
+      <geometry>
+        <mesh
+          filename="file://$(find binocular_laser_profile_scanner)/meshes/rot_table_link.STL" />
       </geometry>
     </collision>
@@ -130,19 +130,19 @@
       <geometry>
         <mesh
-          filename="package://binocular_laser_profile_scanner/meshes/object_link.STL" />
-      </geometry>
-      <material
-        name="">
-        <color
-          rgba="0.792156862745098 0.819607843137255 0.933333333333333 1" />
-      </material>
-    </visual>
-    <collision>
-      <origin
-        xyz="0 0 0"
-        rpy="0 0 0" />
-      <geometry>
-        <mesh
-          filename="package://binocular_laser_profile_scanner/meshes/object_link.STL" />
+          filename="file://$(find binocular_laser_profile_scanner)/meshes/object_link.STL" />
+      </geometry>
+      <material
+        name="">
+        <color
+          rgba="0.792156862745098 0.819607843137255 0.933333333333333 1" />
+      </material>
+    </visual>
+    <collision>
+      <origin
+        xyz="0 0 0"
+        rpy="0 0 0" />
+      <geometry>
+        <mesh
+          filename="file://$(find binocular_laser_profile_scanner)/meshes/object_link.STL" />
       </geometry>
     </collision>
@@ -183,5 +183,5 @@
       <geometry>
         <mesh
-          filename="package://binocular_laser_profile_scanner/meshes/motor_link.STL" />
+          filename="file://$(find binocular_laser_profile_scanner)/meshes/motor_link.STL" />
       </geometry>
       <material
@@ -197,5 +197,5 @@
       <geometry>
         <mesh
-          filename="package://binocular_laser_profile_scanner/meshes/motor_link.STL" />
+          filename="file://$(find binocular_laser_profile_scanner)/meshes/motor_link.STL" />
       </geometry>
     </collision>
@@ -214,5 +214,5 @@
       xyz="0 0 1" />
     <limit
-      lower="0"
+      lower="-0.2"
       upper="3.142"
       effort="1000"
@@ -241,19 +241,19 @@
       <geometry>
         <mesh
-          filename="package://binocular_laser_profile_scanner/meshes/scanner_body_link.STL" />
-      </geometry>
-      <material
-        name="">
-        <color
-          rgba="0.792156862745098 0.819607843137255 0.933333333333333 1" />
-      </material>
-    </visual>
-    <collision>
-      <origin
-        xyz="0 0 0"
-        rpy="0 0 0" />
-      <geometry>
-        <mesh
-          filename="package://binocular_laser_profile_scanner/meshes/scanner_body_link.STL" />
+          filename="file://$(find binocular_laser_profile_scanner)/meshes/scanner_body_link.STL" />
+      </geometry>
+      <material
+        name="">
+        <color
+          rgba="0.792156862745098 0.819607843137255 0.933333333333333 1" />
+      </material>
+    </visual>
+    <collision>
+      <origin
+        xyz="0 0 0"
+        rpy="0 0 0" />
+      <geometry>
+        <mesh
+          filename="file://$(find binocular_laser_profile_scanner)/meshes/scanner_body_link.STL" />
       </geometry>
     </collision>
@@ -294,19 +294,19 @@
       <geometry>
         <mesh
-          filename="package://binocular_laser_profile_scanner/meshes/line_laser_link.STL" />
-      </geometry>
-      <material
-        name="">
-        <color
-          rgba="0.792156862745098 0.819607843137255 0.933333333333333 1" />
-      </material>
-    </visual>
-    <collision>
-      <origin
-        xyz="0 0 0"
-        rpy="0 0 0" />
-      <geometry>
-        <mesh
-          filename="package://binocular_laser_profile_scanner/meshes/line_laser_link.STL" />
+          filename="file://$(find binocular_laser_profile_scanner)/meshes/line_laser_link.STL" />
+      </geometry>
+      <material
+        name="">
+        <color
+          rgba="0.792156862745098 0.819607843137255 0.933333333333333 1" />
+      </material>
+    </visual>
+    <collision>
+      <origin
+        xyz="0 0 0"
+        rpy="0 0 0" />
+      <geometry>
+        <mesh
+          filename="file://$(find binocular_laser_profile_scanner)/meshes/line_laser_link.STL" />
       </geometry>
     </collision>
@@ -352,19 +352,19 @@
       <geometry>
         <mesh
-          filename="package://binocular_laser_profile_scanner/meshes/left_camera_link.STL" />
-      </geometry>
-      <material
-        name="">
-        <color
-          rgba="0.792156862745098 0.819607843137255 0.933333333333333 1" />
-      </material>
-    </visual>
-    <collision>
-      <origin
-        xyz="0 0 0"
-        rpy="0 0 0" />
-      <geometry>
-        <mesh
-          filename="package://binocular_laser_profile_scanner/meshes/left_camera_link.STL" />
+          filename="file://$(find binocular_laser_profile_scanner)/meshes/left_camera_link.STL" />
+      </geometry>
+      <material
+        name="">
+        <color
+          rgba="0.792156862745098 0.819607843137255 0.933333333333333 1" />
+      </material>
+    </visual>
+    <collision>
+      <origin
+        xyz="0 0 0"
+        rpy="0 0 0" />
+      <geometry>
+        <mesh
+          filename="file://$(find binocular_laser_profile_scanner)/meshes/left_camera_link.STL" />
       </geometry>
     </collision>
@@ -405,19 +405,19 @@
       <geometry>
         <mesh
-          filename="package://binocular_laser_profile_scanner/meshes/right_camera_link.STL" />
-      </geometry>
-      <material
-        name="">
-        <color
-          rgba="0.792156862745098 0.819607843137255 0.933333333333333 1" />
-      </material>
-    </visual>
-    <collision>
-      <origin
-        xyz="0 0 0"
-        rpy="0 0 0" />
-      <geometry>
-        <mesh
-          filename="package://binocular_laser_profile_scanner/meshes/right_camera_link.STL" />
+          filename="file://$(find binocular_laser_profile_scanner)/meshes/right_camera_link.STL" />
+      </geometry>
+      <material
+        name="">
+        <color
+          rgba="0.792156862745098 0.819607843137255 0.933333333333333 1" />
+      </material>
+    </visual>
+    <collision>
+      <origin
+        xyz="0 0 0"
+        rpy="0 0 0" />
+      <geometry>
+        <mesh
+          filename="file://$(find binocular_laser_profile_scanner)/meshes/right_camera_link.STL" />
       </geometry>
     </collision>

File: urdf/gazebo_camera.xacro (robot description, xacro)
@@ -2,10 +2,4 @@
 <robot>
   <!--
-    CHANGES
-    * Pixel numbers of image sensor reduced to 600 px x 600 px due to low fps
-    Image Sensor Specs used before
-    Sensor: IMX548
-    Resolution (H x V):2448 px × 2048 px
-    Pixel Size (H x V)	2.74 μm × 2.74 μm
     Image Sensor Specs used currently
     Sensor: Custom
@@ -36,15 +30,13 @@
         <noise>
           <type>gaussian</type>
-          <!-- Noise is sampled independently per pixel on each frame.
-               That pixel's noise value is added to each of its color
-               channels, which at that point lie in the range [0,1]. -->
           <mean>0.0</mean>
           <stddev>0.007</stddev>
         </noise>
       </camera>
-      <plugin name="camera_controller" filename="libgazebo_ros_camera.so">
+      <plugin name="camera_controller_1" filename="libgazebo_ros_camera.so">
         <alwaysOn>true</alwaysOn>
+        <visualize>true</visualize>
         <updateRate>0.0</updateRate>
-        <cameraName>binocular_laser_profile_scanner/left_camera</cameraName>
+        <cameraName>my_package/left_camera</cameraName>
         <imageTopicName>image_raw</imageTopicName>
         <cameraInfoTopicName>camera_info</cameraInfoTopicName>
@@ -76,15 +68,13 @@
         <noise>
           <type>gaussian</type>
-          <!-- Noise is sampled independently per pixel on each frame.
-               That pixel's noise value is added to each of its color
-               channels, which at that point lie in the range [0,1]. -->
           <mean>0.0</mean>
           <stddev>0.007</stddev>
         </noise>
       </camera>
-      <plugin name="camera_controller" filename="libgazebo_ros_camera.so">
+      <plugin name="camera_controller_2" filename="libgazebo_ros_camera.so">
         <alwaysOn>true</alwaysOn>
+        <visualize>true</visualize>
         <updateRate>0.0</updateRate>
-        <cameraName>binocular_laser_profile_scanner/right_camera</cameraName>
+        <cameraName>my_package/right_camera</cameraName>
         <imageTopicName>image_raw</imageTopicName>
         <cameraInfoTopicName>camera_info</cameraInfoTopicName>

File: urdf/gazebo_controller.xacro (robot description, xacro)
@@ -1,30 +1,46 @@
-<?xml version="1.0" encoding="utf-8"?>
+<?xml version="1.0"?>
 <robot>
+  <ros2_control name="GazeboSystem" type="system">
+    <hardware>
+      <plugin>gazebo_ros2_control/GazeboSystem</plugin>
+    </hardware>
+    <joint name="rot_table_joint">
+      <command_interface name="position">
+        <param name="min">0</param>
+        <param name="max">12.568</param>
+      </command_interface>
+      <state_interface name="position">
+        <param name="initial_value">0</param>
+      </state_interface>
+      <state_interface name="velocity"/>
+      <state_interface name="effort"/>
+    </joint>
+    <joint name="motor_joint">
+      <command_interface name="position">
+        <param name="min">-0.2</param>
+        <param name="max">3.142</param>
+      </command_interface>
+      <state_interface name="position">
+        <param name="initial_value">0</param>
+      </state_interface>
+      <state_interface name="velocity"/>
+      <state_interface name="effort"/>
+    </joint>
+    <joint name="line_laser_joint">
+      <command_interface name="position">
+        <param name="min">0</param>
+        <param name="max">0</param>
+      </command_interface>
+      <state_interface name="position">
+        <param name="initial_value">0</param>
+      </state_interface>
+      <state_interface name="velocity"/>
+      <state_interface name="effort"/>
+    </joint>
+  </ros2_control>
   <gazebo>
-    <plugin name="gazebo_ros_control" filename="libgazebo_ros_control.so">
-      <robotNamespace>/binocular_laser_profile_scanner</robotNamespace>
-      <robotSimType>gazebo_ros_control/DefaultRobotHWSim</robotSimType>
+    <plugin filename="libgazebo_ros2_control.so" name="gazebo_ros2_control">
+      <parameters>$(find binocular_laser_profile_scanner)/config/joint_config.yaml</parameters>
     </plugin>
   </gazebo>
-  <!--Position Controllers-->
-  <transmission name="tran1">
-    <type>transmission_interface/SimpleTransmission</type>
-    <joint name="rot_table_joint">
-      <hardwareInterface>hardware_interface/EffortJointInterface</hardwareInterface>
-    </joint>
-    <actuator name="rot_table_motor">
-      <hardwareInterface>hardware_interface/EffortJointInterface</hardwareInterface>
-      <mechanicalReduction>1</mechanicalReduction>
-    </actuator>
-  </transmission>
-  <transmission name="tran2">
-    <type>transmission_interface/SimpleTransmission</type>
-    <joint name="motor_joint">
-      <hardwareInterface>hardware_interface/EffortJointInterface</hardwareInterface>
-    </joint>
-    <actuator name="scanner_angle_motor">
-      <hardwareInterface>hardware_interface/EffortJointInterface</hardwareInterface>
-      <mechanicalReduction>1</mechanicalReduction>
-    </actuator>
-  </transmission>
 </robot>
